Commit message: first version of the urdfs ...

File: velvet_fingers_description/urdf/velvet_fingers.gazebo.xacro (robot description, xacro)
@@ -1,56 +1,26 @@
 <?xml version="1.0"?>
-<robot name="lbr_iiwa" xmlns:xacro="http://www.ros.org/wiki/xacro">
-  <xacro:macro name="lbr_iiwa_gazebo" params="name">
+<robot name="velvet_fingers" xmlns:xacro="http://www.ros.org/wiki/xacro">
+  <xacro:macro name="velvet_fingers_gazebo" params="name">
     <!-- ros_control plugin -->
     <gazebo>
       <plugin name="gazebo_ros_control" filename="libgazebo_ros_control.so">
-	<robotNamespace>/lbr_iiwa</robotNamespace>
+	<robotNamespace>/velvet_fingers</robotNamespace>
       </plugin>
     </gazebo>
-    <!-- Link0 -->
-    <gazebo reference="${name}_link_0">
-      <material>Gazebo/Grey</material>
+    <!-- Palm -->
+    <gazebo reference="${name}_palm">
+      <material>Gazebo/Red</material>
       <mu1>0.2</mu1>
       <mu2>0.2</mu2>
     </gazebo>
-    <!-- Link1 -->
-    <gazebo reference="${name}_link_1">
+    <!-- Right Finger -->
+    <gazebo reference="${name}_right">
       <material>Gazebo/Orange</material>
       <mu1>0.2</mu1>
       <mu2>0.2</mu2>
     </gazebo>
-    <!-- Link2 -->
-    <gazebo reference="${name}_link_2">
+    <!-- Left Finger -->
+    <gazebo reference="${name}_left">
       <material>Gazebo/Orange</material>
-      <mu1>0.2</mu1>
-      <mu2>0.2</mu2>
-    </gazebo>
-    <!-- Link3 -->
-    <gazebo reference="${name}_link_3">
-      <material>Gazebo/Orange</material>
-      <mu1>0.2</mu1>
-      <mu2>0.2</mu2>
-    </gazebo>
-    <!-- Link4 -->
-    <gazebo reference="${name}_link_4">
-      <material>Gazebo/Orange</material>
-      <mu1>0.2</mu1>
-      <mu2>0.2</mu2>
-    </gazebo>
-    <!-- Link5 -->
-    <gazebo reference="${name}_link_5">
-      <material>Gazebo/Orange</material>
-      <mu1>0.2</mu1>
-      <mu2>0.2</mu2>
-    </gazebo>
-    <!-- Link6 -->
-    <gazebo reference="${name}_link_6">
-      <material>Gazebo/Orange</material>
-      <mu1>0.2</mu1>
-      <mu2>0.2</mu2>
-    </gazebo>
-    <!-- Link7 -->
-    <gazebo reference="${name}_link_7">
-      <material>Gazebo/Grey</material>
       <mu1>0.2</mu1>
       <mu2>0.2</mu2>

File: velvet_fingers_description/urdf/velvet_fingers.transmission.xacro (robot description, xacro)
@@ -1,5 +1,5 @@
 <?xml version="1.0"?>
-<robot name="lbr_iiwa" xmlns:xacro="http://www.ros.org/wiki/xacro">
-  <xacro:macro name="lbr_iiwa_transmission" params="name hardware_interface">
+<robot name="velvet_fingers" xmlns:xacro="http://www.ros.org/wiki/xacro">
+  <xacro:macro name="velvet_fingers_transmission" params="name hardware_interface">
     <transmission name="${name}_tran_1">
       <type>transmission_interface/SimpleTransmission</type>
@@ -12,5 +12,5 @@
       </actuator>
     </transmission>
-    <transmission name="${name}_tran_2">
+ <!--  <transmission name="${name}_tran_2">
       <type>transmission_interface/SimpleTransmission</type>
       <joint name="${name}_joint_2">
@@ -21,55 +21,5 @@
 	<mechanicalReduction>1</mechanicalReduction>
       </actuator>
-    </transmission>
-    <transmission name="${name}_tran_3">
-      <type>transmission_interface/SimpleTransmission</type>
-      <joint name="${name}_joint_3">
-	<hardwareInterface>${hardware_interface}</hardwareInterface>
-      </joint>
-      <actuator name="${name}_motor_3">
-	<hardwareInterface>${hardware_interface}</hardwareInterface>
-	<mechanicalReduction>1</mechanicalReduction>
-      </actuator>
-    </transmission>
-    <transmission name="${name}_tran_4">
-      <type>transmission_interface/SimpleTransmission</type>
-      <joint name="${name}_joint_4">
-	<hardwareInterface>${hardware_interface}</hardwareInterface>
-      </joint>
-      <actuator name="${name}_motor_4">
-	<hardwareInterface>${hardware_interface}</hardwareInterface>
-	<mechanicalReduction>1</mechanicalReduction>
-      </actuator>
-    </transmission>
-    <transmission name="${name}_tran_5">
-      <type>transmission_interface/SimpleTransmission</type>
-      <joint name="${name}_joint_5">
-	<hardwareInterface>${hardware_interface}</hardwareInterface>
-      </joint>
-      <actuator name="${name}_motor_5">
-	<hardwareInterface>${hardware_interface}</hardwareInterface>
-	<mechanicalReduction>1</mechanicalReduction>
-      </actuator>
-    </transmission>
-    <transmission name="${name}_tran_6">
-      <type>transmission_interface/SimpleTransmission</type>
-      <joint name="${name}_joint_6">
-	<hardwareInterface>${hardware_interface}</hardwareInterface>
-      </joint>
-      <actuator name="${name}_motor_6">
-	<hardwareInterface>${hardware_interface}</hardwareInterface>
-	<mechanicalReduction>1</mechanicalReduction>
-      </actuator>
-    </transmission>
-    <transmission name="${name}_tran_7">
-      <type>transmission_interface/SimpleTransmission</type>
-      <joint name="${name}_joint_7">
-	<hardwareInterface>${hardware_interface}</hardwareInterface>
-      </joint>
-      <actuator name="${name}_motor_7">
-	<hardwareInterface>${hardware_interface}</hardwareInterface>
-	<mechanicalReduction>1</mechanicalReduction>
-      </actuator>
-    </transmission>
+    </transmission> -->
   </xacro:macro>
 </robot>

File: velvet_fingers_description/urdf/velvet_fingers.urdf.xacro (robot description, xacro)
@@ -1,10 +1,10 @@
 <?xml version="1.0"?>
-<robot name="lbr_iiwa" xmlns:xacro="http://www.ros.org/wiki/xacro">
-  <xacro:include filename="$(find lbr_iiwa_description)/urdf/lbr_iiwa.xacro"/>
+<robot name="velvet_fingers" xmlns:xacro="http://www.ros.org/wiki/xacro">
+  <xacro:include filename="$(find velvet_fingers_description)/urdf/velvet_fingers.xacro"/>
   <!-- Fix to world just for testing -->
   <link name="world"/>
   <!--lbr-->
-  <xacro:lbr_iiwa name="lbr_iiwa" hardware_interface="$(arg prefix)" parent="world">
-    <origin xyz="0 0 0.0" rpy="0 0 0" />
-  </xacro:lbr_iiwa>
+  <xacro:velvet_fingers name="velvet_fingers" hardware_interface="$(arg prefix)" parent="world">
+    <origin xyz="0 0 0.5" rpy="0 0 0" />
+  </xacro:velvet_fingers>
 </robot>

File: velvet_fingers_description/urdf/velvet_fingers.xacro (robot description, xacro)
@@ -1,53 +1,53 @@
 <?xml version="1.0"?>
-<robot name="lbr_iiwa" xmlns:xacro="http://www.ros.org/wiki/xacro">
+<robot name="velvet_fingers" xmlns:xacro="http://www.ros.org/wiki/xacro">
   <!-- Import all Gazebo-customization elements, including Gazebo colors -->
-  <xacro:include filename="$(find lbr_iiwa_description)/urdf/lbr_iiwa.gazebo.xacro" />
+  <xacro:include filename="$(find velvet_fingers_description)/urdf/velvet_fingers.gazebo.xacro" />
   <!-- Import Rviz colors -->
-  <xacro:include filename="$(find lbr_iiwa_description)/urdf/materials.xacro" />
+  <xacro:include filename="$(find velvet_fingers_description)/urdf/materials.xacro" />
   <!-- Import Transmissions -->
-  <xacro:include filename="$(find lbr_iiwa_description)/urdf/lbr_iiwa.transmission.xacro" />
+  <xacro:include filename="$(find velvet_fingers_description)/urdf/velvet_fingers.transmission.xacro" />
   <!-- Include Utilities -->
-  <xacro:include filename="$(find lbr_iiwa_description)/urdf/utilities.xacro" />
+  <xacro:include filename="$(find velvet_fingers_description)/urdf/utilities.xacro" />
   <!-- some constants -->
  <!-- <xacro:property name="safety_controller_k_pos" value="100" />
   <xacro:property name="safety_controller_k_vel" value="2" /> -->
   <xacro:property name="joint_damping" value="0.5" />
-  <xacro:property name="max_effort" value="300"/>
+  <xacro:property name="max_effort" value="100"/>
   <xacro:property name="max_velocity" value="10"/>
-  <xacro:macro name="lbr_iiwa" params="parent name hardware_interface *origin">
-    <!--joint between {parent} and link_0-->
+  <xacro:macro name="velvet_fingers" params="parent name hardware_interface *origin">
+    <!--joint between {parent} and palm -->
     <joint name="${parent}_joint" type="fixed">
       <insert_block name="origin"/>
       <parent link="${parent}"/>
-      <child link="${name}_link_0"/>
+      <child link="${name}_palm"/>
     </joint>
-    <link name="${name}_link_0">
+    <link name="${name}_palm">
       <inertial>
-        <origin xyz="-0.1 0 0.07" rpy="0 0 0"/>
-        <mass value="5"/>
-        <inertia ixx="0.05"  ixy="0"  ixz="0" iyy="0.06" iyz="0" izz="0.03" />
+        <origin xyz="0.04 0.0 -0.01" rpy="0 0 0"/>
+        <mass value="0.8"/>
+        <inertia ixx="0.003"  ixy="0"  ixz="0" iyy="0.005" iyz="0" izz="0.004" />
       </inertial>
       <visual>
         <origin xyz="0 0 0" rpy="0 0 0"/>
         <geometry>
-          <mesh filename="package://lbr_iiwa_description/meshes/link_0.stl"/>
+          <mesh filename="package://velvet_fingers_description/meshes/velvet_fingers_palm.stl"/>
         </geometry>
-        <material name="Grey"/>
+        <material name="Red"/>
       </visual>
       <collision>
         <origin xyz="0 0 0" rpy="0 0 0"/>
         <geometry>
-          <mesh filename="package://lbr_iiwa_description/meshes/coarse/link_0.stl"/>
+          <mesh filename="package://velvet_fingers_description/meshes/velvet_fingers_palm.stl"/>
         </geometry>
-        <material name="Grey"/>
+        <material name="Red"/>
       </collision>
     </link>
-    <!-- joint between link_0 and link_1 -->
+    <!-- joint between palm and right finger -->
     <joint name="${name}_joint_1" type="revolute">
-      <parent link="${name}_link_0"/>
-      <child link="${name}_link_1"/>
-      <origin xyz="0 0 0.1575" rpy="0 0 0"/>
+      <parent link="${name}_palm"/>
+      <child link="${name}_right"/>
+      <origin xyz="0.121 -0.016 0.0" rpy="0 0 ${-PI / 2}"/>
       <axis xyz="0 0 1"/>
-      <limit lower="${-170 * PI / 180}" upper="${170 * PI / 180}"
+      <limit lower="${0 * PI / 180}" upper="${90 * PI / 180}"
              effort="${max_effort}" velocity="${max_velocity}" />
       <!--   <safety_controller soft_lower_limit="${-168 * M_PI / 180}"
@@ -57,14 +57,14 @@
       <dynamics damping="${joint_damping}"/>
     </joint>
-    <link name="${name}_link_1">
+    <link name="${name}_right">
       <inertial>
-        <origin xyz="0 -0.03 0.12" rpy="0 0 0"/>
-        <mass value="4"/>
-        <inertia ixx="0.1"  ixy="0"  ixz="0" iyy="0.09" iyz="0" izz="0.02" />
+        <origin xyz="0.01 0 0" rpy="0 0 0"/>
+        <mass value="0.5"/>
+        <inertia ixx="0.001"  ixy="0"  ixz="0" iyy="0.001" iyz="0" izz="0.001" />
       </inertial>
       <visual>
         <origin xyz="0 0 0" rpy="0 0 0"/>
         <geometry>
-          <mesh filename="package://lbr_iiwa_description/meshes/link_1.stl"/>
+          <mesh filename="package://velvet_fingers_description/meshes/velvet_fingers_right.stl"/>
         </geometry>
         <material name="Orange"/>
@@ -73,33 +73,34 @@
         <origin xyz="0 0 0" rpy="0 0 0"/>
         <geometry>
-          <mesh filename="package://lbr_iiwa_description/meshes/coarse/link_1.stl"/>
+          <mesh filename="package://velvet_fingers_description/meshes/velvet_fingers_right.stl"/>
         </geometry>
         <material name="Orange"/>
       </collision>
     </link>
-    <!-- joint between link_1 and link_2 -->
+    <!-- joint between palm and left finger -->
     <joint name="${name}_joint_2" type="revolute">
-      <parent link="${name}_link_1"/>
-      <child link="${name}_link_2"/>
-      <origin xyz="0 0 0.2025" rpy="0 0 0"/>
-      <axis xyz="0 1 0"/>
-      <limit lower="${-120 * PI / 180}" upper="${120 * PI / 180}"
+      <parent link="${name}_palm"/>
+      <child link="${name}_left"/>
+      <origin xyz="0.121 0.016 0.0" rpy="${PI} 0 ${PI / 2}"/>
+      <axis xyz="0 0 1"/>
+      <limit lower="${0 * PI / 180}" upper="${90 * PI / 180}"
              effort="${max_effort}" velocity="${max_velocity}" />
-      <!-- <safety_controller soft_lower_limit="${-118 * PI / 180}"
-           soft_upper_limit="${118 * PI / 180}"
+      <!--   <safety_controller soft_lower_limit="${-168 * M_PI / 180}"
+           soft_upper_limit="${168 * M_PI / 180}"
            k_position="${safety_controller_k_pos}"
            k_velocity="${safety_controller_k_vel}"/> -->
       <dynamics damping="${joint_damping}"/>
+      <mimic joint="${name}_joint_1"/>
     </joint>
-    <link name="${name}_link_2">
+    <link name="${name}_left">
       <inertial>
-        <origin xyz="0 0.04 0.06" rpy="0 0 0"/>
-        <mass value="4"/>
-        <inertia ixx="0.05"  ixy="0"  ixz="0" iyy="0.04" iyz="0" izz="0.02" />
+        <origin xyz="0.01 0 0" rpy="0 0 0"/>
+        <mass value="0.5"/>
+        <inertia ixx="0.001"  ixy="0"  ixz="0" iyy="0.001" iyz="0" izz="0.001" />
       </inertial>
       <visual>
         <origin xyz="0 0 0" rpy="0 0 0"/>
         <geometry>
-          <mesh filename="package://lbr_iiwa_description/meshes/link_2.stl"/>
+          <mesh filename="package://velvet_fingers_description/meshes/velvet_fingers_left.stl"/>
         </geometry>
         <material name="Orange"/>
@@ -108,187 +109,12 @@
         <origin xyz="0 0 0" rpy="0 0 0"/>
         <geometry>
-          <mesh filename="package://lbr_iiwa_description/meshes/coarse/link_2.stl"/>
+          <mesh filename="package://velvet_fingers_description/meshes/velvet_fingers_left.stl"/>
         </geometry>
         <material name="Orange"/>
       </collision>
     </link>
-    <!-- joint between link_2 and link_3 -->
-    <joint name="${name}_joint_3" type="revolute">
-      <parent link="${name}_link_2"/>
-      <child link="${name}_link_3"/>
-      <origin xyz="0 0 0.2045" rpy="0 0 0"/>
-      <axis xyz="0 0 1"/>
-      <limit lower="${-170 * PI / 180}" upper="${170 * PI / 180}"
-             effort="${max_effort}" velocity="${max_velocity}" />
-      <!-- <safety_controller soft_lower_limit="${-118 * PI / 180}"
-           soft_upper_limit="${118 * PI / 180}"
-           k_position="${safety_controller_k_pos}"
-           k_velocity="${safety_controller_k_vel}"/> -->
-      <dynamics damping="${joint_damping}"/>
-    </joint>
-    <link name="${name}_link_3">
-      <inertial>
-        <origin xyz="0 0.03 0.13" rpy="0 0 0"/>
-        <mass value="3"/>
-        <inertia ixx="0.08"  ixy="0"  ixz="0" iyy="0.07" iyz="0" izz="0.01" />
-      </inertial>
-      <visual>
-        <origin xyz="0 0 0" rpy="0 0 0"/>
-        <geometry>
-          <mesh filename="package://lbr_iiwa_description/meshes/link_3.stl"/>
-        </geometry>
-        <material name="Orange"/>
-      </visual>
-      <collision>
-        <origin xyz="0 0 0" rpy="0 0 0"/>
-        <geometry>
-          <mesh filename="package://lbr_iiwa_description/meshes/coarse/link_3.stl"/>
-        </geometry>
-        <material name="Orange"/>
-      </collision>
-    </link>
-   <!-- joint between link_3 and link_4 -->
-    <joint name="${name}_joint_4" type="revolute">
-      <parent link="${name}_link_3"/>
-      <child link="${name}_link_4"/>
-      <origin xyz="0 0 0.2155" rpy="0 0 0"/>
-      <axis xyz="0 1 0"/>
-      <limit lower="${-120 * PI / 180}" upper="${120 * PI / 180}"
-             effort="${max_effort}" velocity="${max_velocity}" />
-      <!-- <safety_controller soft_lower_limit="${-118 * PI / 180}"
-           soft_upper_limit="${118 * PI / 180}"
-           k_position="${safety_controller_k_pos}"
-           k_velocity="${safety_controller_k_vel}"/> -->
-      <dynamics damping="${joint_damping}"/>
-    </joint>
-    <link name="${name}_link_4">
-      <inertial>
-        <origin xyz="0 -0.03 0.07" rpy="0 0 0"/>
-        <mass value="2.5"/>
-        <inertia ixx="0.03"  ixy="0"  ixz="0" iyy="0.03" iyz="0" izz="0.01" />
-      </inertial>
-      <visual>
-        <origin xyz="0 0 0" rpy="0 0 0"/>
-        <geometry>
-          <mesh filename="package://lbr_iiwa_description/meshes/link_4.stl"/>
-        </geometry>
-        <material name="Orange"/>
-      </visual>
-      <collision>
-        <origin xyz="0 0 0" rpy="0 0 0"/>
-        <geometry>
-          <mesh filename="package://lbr_iiwa_description/meshes/coarse/link_4.stl"/>
-        </geometry>
-        <material name="Orange"/>
-      </collision>
-    </link>
-    <!-- joint between link_4 and link_5 -->
-    <joint name="${name}_joint_5" type="revolute">
-      <parent link="${name}_link_4"/>
-      <child link="${name}_link_5"/>
-      <origin xyz="0 0 0.1845" rpy="0 0 0"/>
-      <axis xyz="0 0 1"/>
-      <limit lower="${-170 * PI / 180}" upper="${170 * PI / 180}"
-             effort="${max_effort}" velocity="${max_velocity}" />
-      <!-- <safety_controller soft_lower_limit="${-118 * PI / 180}"
-           soft_upper_limit="${118 * PI / 180}"
-           k_position="${safety_controller_k_pos}"
-           k_velocity="${safety_controller_k_vel}"/> -->
-      <dynamics damping="${joint_damping}"/>
-    </joint>
-    <link name="${name}_link_5">
-      <inertial>
-        <origin xyz="0 -0.02 0.08" rpy="0 0 0"/>
-        <mass value="1.7"/>
-        <inertia ixx="0.02"  ixy="0"  ixz="0" iyy="0.02" iyz="0" izz="0.01" />
-      </inertial>
-      <visual>
-        <origin xyz="0 0 0" rpy="0 0 0"/>
-        <geometry>
-          <mesh filename="package://lbr_iiwa_description/meshes/link_5.stl"/>
-        </geometry>
-        <material name="Orange"/>
-      </visual>
-      <collision>
-        <origin xyz="0 0 0" rpy="0 0 0"/>
-        <geometry>
-          <mesh filename="package://lbr_iiwa_description/meshes/coarse/link_5.stl"/>
-        </geometry>
-        <material name="Orange"/>
-      </collision>
-    </link>
- <!-- joint between link_5 and link_6 -->
-    <joint name="${name}_joint_6" type="revolute">
-      <parent link="${name}_link_5"/>
-      <child link="${name}_link_6"/>
-      <origin xyz="0 -0.0607 0.2155" rpy="0 0 0"/>
-      <axis xyz="0 1 0"/>
-      <limit lower="${-120 * PI / 180}" upper="${120 * PI / 180}"
-             effort="${max_effort}" velocity="${max_velocity}" />
-      <!-- <safety_controller soft_lower_limit="${-118 * PI / 180}"
-           soft_upper_limit="${118 * PI / 180}"
-           k_position="${safety_controller_k_pos}"
-           k_velocity="${safety_controller_k_vel}"/> -->
-      <dynamics damping="${joint_damping}"/>
-    </joint>
-    <link name="${name}_link_6">
-      <inertial>
-        <origin xyz="0 0.06 0" rpy="0 0 0"/>
-        <mass value="1.8"/>
-        <inertia ixx="0.01"  ixy="0"  ixz="0" iyy="0.001" iyz="0" izz="0.01" />
-      </inertial>
-      <visual>
-        <origin xyz="0 0 0" rpy="0 0 0"/>
-        <geometry>
-          <mesh filename="package://lbr_iiwa_description/meshes/link_6.stl"/>
-        </geometry>
-        <material name="Orange"/>
-      </visual>
-      <collision>
-        <origin xyz="0 0 0" rpy="0 0 0"/>
-        <geometry>
-          <mesh filename="package://lbr_iiwa_description/meshes/coarse/link_6.stl"/>
-        </geometry>
-        <material name="Orange"/>
-      </collision>
-    </link>
- <!-- joint between link_6 and link_7 -->
-    <joint name="${name}_joint_7" type="revolute">
-      <parent link="${name}_link_6"/>
-      <child link="${name}_link_7"/>
-      <origin xyz="0 0.0607 0.0809" rpy="0 0 0"/>
-      <axis xyz="0 0 1"/>
-      <limit lower="${-175 * PI / 180}" upper="${175 * PI / 180}"
-             effort="${max_effort}" velocity="${max_velocity}" />
-      <!-- <safety_controller soft_lower_limit="${-118 * PI / 180}"
-           soft_upper_limit="${118 * PI / 180}"
-           k_position="${safety_controller_k_pos}"
-           k_velocity="${safety_controller_k_vel}"/> -->
-      <dynamics damping="${joint_damping}"/>
-    </joint>
-    <link name="${name}_link_7">
-      <inertial>
-        <origin xyz="0 0 0.02" rpy="0 0 0"/>
-        <mass value="0.3"/>
-        <inertia ixx="0.001"  ixy="0"  ixz="0" iyy="0.001" iyz="0" izz="0.001" />
-      </inertial>
-      <visual>
-        <origin xyz="0 0 0" rpy="0 0 0"/>
-        <geometry>
-          <mesh filename="package://lbr_iiwa_description/meshes/link_7.stl"/>
-        </geometry>
-        <material name="Grey"/>
-      </visual>
-      <collision>
-        <origin xyz="0 0 0" rpy="0 0 0"/>
-        <geometry>
-          <mesh filename="package://lbr_iiwa_description/meshes/coarse/link_7.stl"/>
-        </geometry>
-        <material name="Grey"/>
-      </collision>
-    </link>
     <!--Extensions -->
-    <xacro:lbr_iiwa_gazebo name="${name}" />
-    <xacro:lbr_iiwa_transmission name="${name}" hardware_interface="${hardware_interface}"/>
+    <xacro:velvet_fingers_gazebo name="${name}" />
+    <xacro:velvet_fingers_transmission name="${name}" hardware_interface="${hardware_interface}"/>
   </xacro:macro>
 </robot>

Commit message: velvet_fingers_control: added gazebo mimic plugin for the gripper o/c joint

File: velvet_fingers_description/urdf/velvet_fingers.gazebo.xacro (robot description, xacro)
@@ -6,4 +6,12 @@
       <plugin name="gazebo_ros_control" filename="libgazebo_ros_control.so">
 	<robotNamespace>/velvet_fingers</robotNamespace>
+      </plugin>
+    </gazebo>
+   <!-- Plugin for the mimic o/c joint - AFAIK, that shouldn't be necessary any more starting with Gazebo 3.0 -->
+    <gazebo>
+      <plugin name="mimic_plugin" filename="libgazebo_mimic_plugin.so">
+       <joint>${name}_joint_1</joint>
+        <mimicJoint>${name}_joint_2</mimicJoint>
+        <multiplier>1.0</multiplier>
       </plugin>
     </gazebo>
