Commit message: fixed urdf colors

File: velvet_fingers_description/urdf/materials.xacro (robot description, xacro)
@@ -1,26 +1,26 @@
 <?xml version="1.0"?>
 <robot name="apple" xmlns:xacro="http://www.ros.org/wiki/xacro">
-  <material name="Black">
+  <material name="VELVET_FINGERS/Black">
     <color rgba="0.0 0.0 0.0 1.0"/>
   </material>
-  <material name="Blue">
+  <material name="VELVET_FINGERS/Blue">
     <color rgba="0.0 0.0 0.8 1.0"/>
   </material>
-  <material name="Green">
+  <material name="VELVET_FINGERS/Green">
     <color rgba="0.0 0.8 0.0 1.0"/>
   </material>
-  <material name="Grey">
+  <material name="VELVET_FINGERS/Grey">
     <color rgba="0.2 0.2 0.2 1.0"/>
   </material>
-  <material name="Orange">
+  <material name="VELVET_FINGERS/Orange">
     <color rgba="${255/255} ${108/255} ${10/255} 1.0"/>
   </material>
-  <material name="Brown">
+  <material name="VELVET_FINGERS/Brown">
     <color rgba="${222/255} ${207/255} ${195/255} 1.0"/>
   </material>
-  <material name="Red">
+  <material name="VELVET_FINGERS/Red">
     <color rgba="0.8 0.0 0.0 1.0"/>
   </material>
-  <material name="White">
+  <material name="VELVET_FINGERS/White">
     <color rgba="1.0 1.0 1.0 1.0"/>
   </material>

File: velvet_fingers_description/urdf/velvet_fingers.urdf.xacro (robot description, xacro)
@@ -1,6 +1,4 @@
 <?xml version="1.0"?>
 <robot name="velvet_fingers" xmlns:xacro="http://www.ros.org/wiki/xacro">
-  <!-- Import Rviz colors -->
-  <xacro:include filename="$(find velvet_fingers_description)/urdf/materials.xacro" />
   <!-- Import the velvet fingers macro -->
   <xacro:include filename="$(find velvet_fingers_description)/urdf/velvet_fingers.xacro"/>

File: velvet_fingers_description/urdf/velvet_fingers.xacro (robot description, xacro)
@@ -7,4 +7,6 @@
   <!-- Include Utilities -->
   <xacro:include filename="$(find velvet_fingers_description)/urdf/utilities.xacro" />
+  <!-- Import Rviz colors -->
+  <xacro:include filename="$(find velvet_fingers_description)/urdf/materials.xacro" />
   <!-- some constants -->
  <!-- <xacro:property name="safety_controller_k_pos" value="100" />
@@ -31,5 +33,5 @@
           <mesh filename="package://velvet_fingers_description/meshes/velvet_fingers_palm.stl"/>
         </geometry>
-        <material name="Red"/>
+        <material name="VELVET_FINGERS/Red"/>
       </visual>
       <collision>
@@ -38,5 +40,5 @@
           <mesh filename="package://velvet_fingers_description/meshes/velvet_fingers_palm.stl"/>
         </geometry>
-        <material name="Red"/>
+        <material name="VELVET_FINGERS/Red"/>
       </collision>
     </link>
@@ -66,5 +68,5 @@
           <mesh filename="package://velvet_fingers_description/meshes/velvet_fingers_right.stl"/>
         </geometry>
-        <material name="Orange"/>
+        <material name="VELVET_FINGERS/Orange"/>
       </visual>
       <collision>
@@ -73,5 +75,5 @@
           <mesh filename="package://velvet_fingers_description/meshes/velvet_fingers_right.stl"/>
         </geometry>
-        <material name="Orange"/>
+        <material name="VELVET_FINGERS/Orange"/>
       </collision>
     </link>
@@ -102,5 +104,5 @@
           <mesh filename="package://velvet_fingers_description/meshes/velvet_fingers_left.stl"/>
         </geometry>
-        <material name="Orange"/>
+        <material name="VELVET_FINGERS/Orange"/>
       </visual>
       <collision>
@@ -109,5 +111,5 @@
           <mesh filename="package://velvet_fingers_description/meshes/velvet_fingers_left.stl"/>
         </geometry>
-        <material name="Orange"/>
+        <material name="VELVET_FINGERS/Orange"/>
       </collision>
     </link>
